File: KiCAD/ESPTINY86_Mixtape_version2.kicad_pcb (KiCad board)
At the start: 2 copper layers, 99 x 64.8 mm, 34 parts, among them IC1 4051, IC2 DAC7513_DCN, J1 Bat_EXT, SW1 SW_SPST, SW2 SW_Push, SW3 SW_Push, U1 WeMos_mini

Commit message: adding parts s placement
Parts:
- SW2, SW3: footprint ESPTINY86_MixtapePCB:SW_PUSH-12mm_3D_SMD-top -> ESPTINY86_MixtapePCB:SW_PUSH-8mm_SMD
Routing:
- net GND: track 217.5 -> 206.6 mm
- net Net-(R5-Pad1): track 15.8 -> 9.70 mm
- net Net-(R3-Pad1): track 19.1 -> 13.4 mm
- net +3V3: vias 15 -> 14
