File: KiCAD/ESPTINY86_Mixtape_version2.sch (KiCad schematic (older format))
At the start: 30 parts, among them IC1 4051, IC2 DAC7513_DCN, J1 Bat_EXT, SW1 SW_SPST, SW2 SW_Push, SW3 SW_Push, U1 WeMos_mini

Commit message: fixing the schematic
Parts:
- removed IC2: DAC7513_DCN, ESPTINY86_MixtapePCB:SOIC-8_3.9x4.9mm_Pitch1.27mm, symbol DAC7513_DCN
- added IC2: PT8211, symbol PT8211
Connections:
- net labels removed: PDS
- wire segments 110 -> 111
Changed lines of the file:
@@
-$EndComp
-$Comp
-L DAC7513_DCN IC2
-U 1 1 5B59CC9F
-P 3800 6650
-F 0 "IC2" H 3700 7125 50  0000 R CNN
-F 1 "DAC7513_DCN" H 3700 7050 50  0000 R CNN
-F 2 "ESPTINY86_MixtapePCB:SOIC-8_3.9x4.9mm_Pitch1.27mm" H 3850 6250 50  0001 L CNN
-F 3 "" H 3800 6650 50  0001 C CNN
-	1    3800 6650
-	0    -1   -1   0
 $EndComp
 $Comp
@@
 L GND #PWR019
 U 1 1 5B5A1941
-P 3300 6650
-F 0 "#PWR019" H 3300 6400 50  0001 C CNN
-F 1 "GND" H 3300 6500 50  0000 C CNN
-F 2 "" H 3300 6650 50  0001 C CNN
-F 3 "" H 3300 6650 50  0001 C CNN
-	1    3300 6650
+P 3150 6650
+F 0 "#PWR019" H 3150 6400 50  0001 C CNN
+F 1 "GND" H 3150 6500 50  0000 C CNN
+F 2 "" H 3150 6650 50  0001 C CNN
+F 3 "" H 3150 6650 50  0001 C CNN
+	1    3150 6650
 	1    0    0    -1
 $EndComp
@@
 	0    1    1    0
 $EndComp
-Text Label 4600 6200 0    60   ~ 0
-PDS
 $Comp
 L WeMos_mini U1
@@
 Wire Wire Line
 	4400 6650 4400 6600
+$Comp
+L PT8211 IC2
+U 1 1 5C12ED64
+P 3800 6650
+F 0 "IC2" H 3700 7125 50  0000 R CNN
+F 1 "PT8211" H 3700 7050 50  0000 R CNN
+F 2 "" H 3850 6250 50  0001 L CNN
+F 3 "" H 3800 6650 50  0001 C CNN
+	1    3800 6650
+	0    -1   -1   0
+$EndComp
+Wire Wire Line
+	3300 6650 3150 6650
 $EndSCHEMATC

Commit message: adding parts s placement
Connections:
- wire segments 111 -> 116
Changed lines of the file:
@@
 	4300 4950 3900 4950
 Wire Wire Line
-	3900 4950 3900 4000
-Wire Wire Line
-	3900 4000 2950 4000
+	3900 4950 3900 4250
+Wire Wire Line
+	3900 4250 2950 4250
 Wire Wire Line
 	4300 5050 3800 5050
 Wire Wire Line
-	3800 5050 3800 3900
-Wire Wire Line
-	3800 3900 2800 3900
+	3800 5050 3800 4350
+Wire Wire Line
+	3800 4350 2800 4350
 Wire Wire Line
 	4300 3850 4250 3850
@@
 	7150 3850 6950 3850
 Wire Wire Line
-	5700 4950 5700 5200
+	5700 4950 5700 5150
+Wire Wire Line
+	5700 5150 5700 5200
 Wire Wire Line
 	4300 4750 4300 5150
@@
 	6750 1250 6750 1400
 Wire Wire Line
-	8450 3850 8450 4450
+	8450 3850 8450 4050
+Wire Wire Line
+	8450 4050 8450 4450
 Wire Wire Line
 	5000 3800 5000 3700
@@
 	1550 4250 1700 4250
 Wire Wire Line
-	2950 4000 2950 4200
-Wire Wire Line
-	2950 4200 2850 4200
-Wire Wire Line
-	2850 4200 2850 4250
+	2950 4250 2850 4250
+Wire Wire Line
+	2850 4250 2850 4250
 Wire Wire Line
 	2850 4250 2700 4250
 Wire Wire Line
-	2800 3900 2800 4350
+	2800 4350 2800 4350
 Wire Wire Line
 	2800 4350 2700 4350
@@
 	2700 4750 2700 5000
 Wire Wire Line
-	3700 1950 3850 1950
+	3700 1950 3800 1950
+Wire Wire Line
+	3800 1950 3850 1950
 Wire Wire Line
 	2700 4550 3550 4550
@@
 	1050 4150 1700 4150
 Wire Wire Line
-	3550 4550 3550 5700
+	3550 4550 3550 5300
+Wire Wire Line
+	3550 5300 3550 5700
 $Comp
 L LED D1
@@
 	5700 2450 5550 2450
 Wire Wire Line
-	5150 2100 5150 2450
+	5150 2100 5150 2250
+Wire Wire Line
+	5150 2250 5150 2450
 Wire Wire Line
 	5150 2450 5250 2450
 Wire Wire Line
-	5000 2250 7100 2250
+	5000 2250 5150 2250
+Wire Wire Line
+	5150 2250 7100 2250
 Wire Wire Line
 	7100 2250 7100 2350
